Commit message: Add wrist camera and teleoperation node

File: urdf/arm.urdf.xacro (robot description, xacro)
@@ -13,3 +13,11 @@
     <!-- Camera - commentare per escludere dal modello -->
     <xacro:include filename="armando_camera.urdf.xacro"/>
+    <!-- Camera 1 (Fissa): usa tutti i valori di default -->
+    <xacro:camera_sensor prefix="camera" parent_link="camera_mount" topic_name="camera">
+        <origin xyz="0 0 0" rpy="0 0 0"/>
+    </xacro:camera_sensor>
+    <!-- Camera 2 (Wrist): usa i default per risoluzione e framerate -->
+    <xacro:camera_sensor prefix="wrist_camera" parent_link="crawer_base" topic_name="wrist_camera">
+        <origin xyz="0 0 0" rpy="0 -1.5708 0"/>
+    </xacro:camera_sensor>
 </robot>

File: urdf/armando_camera.urdf.xacro (robot description, xacro)
@@ -1,43 +1,67 @@
 <?xml version="1.0"?>
 <robot xmlns:xacro="http://www.ros.org/wiki/xacro">
-    <joint name="camera_joint" type="fixed">
-        <parent link="camera_mount"/>
-        <child link="camera_link"/>
-        <origin xyz="0.0 0.0 0.0" rpy="0 0 0"/>
-    </joint>
-    <link name="camera_link">
-        <visual>
-            <geometry>
-                <box size="0.01 0.03 0.03"/>
-            </geometry>
-            <material name="red"/>
-        </visual>
-    </link>
-    <joint name="camera_optical_joint" type="fixed">
-        <parent link="camera_link"/>
-        <child link="camera_optical_frame"/>
-        <origin xyz="0 0 0" rpy="-1.57079632679 0 -1.57079632679"/>
-    </joint>
-    <link name="camera_optical_frame"/>
-    <!-- ==== Plugin Sensore ==== -->
-    <gazebo reference="camera_link">
-        <sensor name="camera" type="camera">
-            <camera>
-                <horizontal_fov>1.047</horizontal_fov>
-                <image>
-                    <width>1920</width>
-                    <height>1080</height>
-                </image>
-                <clip>
-                    <near>0.1</near>
-                    <far>5</far>
-                </clip>
-            </camera>
-            <always_on>1</always_on>
-            <update_rate>30</update_rate>
-            <visualize>true</visualize>
-            <topic>camera</topic>
-            <gz_frame_id>camera_optical_frame</gz_frame_id>
-        </sensor>
-    </gazebo>
+    <!-- ========================================================================= -->
+    <!-- METODO 2: Macro con valori di default facoltativi (sintassi :=)           -->
+    <!-- Se width, height, update_rate o fov non vengono passati, si usano         -->
+    <!-- i valori predefiniti (1080p, 30 FPS, FOV 60deg).                          -->
+    <!-- ========================================================================= -->
+    <xacro:macro name="camera_sensor"
+                 params="prefix
+                         parent_link
+                         topic_name
+                         width:=1920
+                         height:=1080
+                         update_rate:=30
+                         fov:=1.047
+                         *origin">
+        <joint name="${prefix}_joint" type="fixed">
+            <parent link="${parent_link}"/>
+            <child link="${prefix}_link"/>
+            <xacro:insert_block name="origin"/>
+        </joint>
+        <link name="${prefix}_link">
+            <visual>
+                <geometry>
+                    <box size="0.01 0.03 0.03"/>
+                </geometry>
+                <material name="red"/>
+            </visual>
+            <!--<collision>
+                <geometry>
+                    <box size="0.01 0.03 0.03"/>
+                </geometry>
+            </collision>
+            <inertial>
+                <mass value="0.05"/>
+                <origin xyz="0 0 0" rpy="0 0 0"/>
+                <inertia ixx="1e-5" ixy="0.0" ixz="0.0" iyy="1e-5" iyz="0.0" izz="1e-5"/>
+            </inertial> -->
+        </link>
+        <joint name="${prefix}_optical_joint" type="fixed">
+            <parent link="${prefix}_link"/>
+            <child link="${prefix}_optical_frame"/>
+            <origin xyz="0 0 0" rpy="-1.57079632679 0 -1.57079632679"/>
+        </joint>
+        <link name="${prefix}_optical_frame"/>
+        <gazebo reference="${prefix}_link">
+            <sensor name="${prefix}" type="camera">
+                <camera>
+                    <horizontal_fov>${fov}</horizontal_fov>
+                    <image>
+                        <width>${width}</width>
+                        <height>${height}</height>
+                    </image>
+                    <clip>
+                        <near>0.1</near>
+                        <far>5.0</far>
+                    </clip>
+                </camera>
+                <always_on>1</always_on>
+                <update_rate>${update_rate}</update_rate>
+                <visualize>true</visualize>
+                <topic>${topic_name}</topic>
+                <gz_frame_id>${prefix}_optical_frame</gz_frame_id>
+            </sensor>
+        </gazebo>
+    </xacro:macro>
 </robot>
